File: 1-baseboard/TentaLab/tentalab.kicad_pcb (KiCad board)
At the start: 4 copper layers, 171.4 x 243.8 mm, 480 parts, among them J1 USB-A_USB-303WSD-BRY, J10 Micro_SD_Card, J11 RPI_HEADER, J12 RPI_OPTIONS, J13 RJ45_HC612601A-M893-A, J14 PCIe, J15 PCIe, J16 12V ATX, J17 JTAG_0, J18 JTAG_0, J19 JTAG_0, J2 JTAG_UPSTREAM, J20 Jack-DC, J21 FPGA_RST_nPRSNT, J22 PCIe, J23 RPi UART, J24 JTAG_0, J25 JTAG_SKIP_0, J26 JTAG_SKIP_0, J27 JTAG_SKIP_0, J28 JTAG_SKIP_0, J29 Conn_01x22_Female, J3 CM5_1-100_3mm-stack, J30 Conn_01x22_Female, J31 SFP+, J32 SFP+, J33 SFP+, J34 SFP+, J35 SFP+, J36 SFP+, J37 PCIe, J38 SFP+, J39 SFP+, J4 CM5_101-200_3mm-stack, J5 HDMI_A, J6 Conn_Coaxial_Small, J7 HDMI_A, J8 Conn_01x04, J9 RPi USB2, SW1 PWR_BTN, U1 AP22615AWU-7, U12 RT9742SNGV, U2 PI7C9X2G608ELBZXAE, U3 TPS62821DLC, U4 M93C86, U5 CH330N, U6 TPS563200, U7 AP22615AWU-7

Commit message: baseboard sch with qsfp, layout in progress
Parts:
- removed C107, C109, C114, C116, C117, C118, C125, C126, C127, C128, C135, C136, C137, C138, C145, C146, C147, C148, C155, C156, C157, C158, C165, C166, C168, C169, C176, C177, C178, C179, C186, C187: 100n, Capacitor_SMD:C_0402_1005Metric
- removed C108, C115, C121, C122, C131, C132, C141, C142, C151, C152, C161, C162, C172, C173, C182, C183: 22u, Capacitor_SMD:C_0603_1608Metric_Pad1.08x0.95mm_HandSolder
- removed C110, C111, C119, C120, C129, C130, C139, C140, C149, C150, C159, C160, C170, C171, C180, C181: 100nF, Capacitor_SMD:C_0402_1005Metric
- removed C112, C113, C123, C124, C133, C134, C143, C144, C153, C154, C163, C164, C174, C175, C184, C185: 22uF, Capacitor_SMD:C_0603_1608Metric
- removed D28, D29, D30, D31, D32, D33, D34, D35: LED-R-0603_KT-0603R, cm5-module-Library:LED_0603_1608Metric_R
- removed J31, J32, J33, J34, J35, J36, J38, J39: SFP+, Connector:Connector_SFP_and_Cage
- removed L10, L11, L12, L13, L14, L15, L16, L17, L18, L19, L20, L21, L6, L7, L8, L9: 470nH, Inductor_SMD:L_0603_1608Metric_Pad1.05x0.95mm_HandSolder
- removed R172, R173, R183, R184, R191, R192, R193, R194, R204, R205, R206, R207, R217, R218, R219, R220, R230, R231, R232, R233, R243, R244, R245, R246, R256, R257, R258, R259, R269, R270, R271, R272: R-10k-0402, Resistor_SMD:R_0402_1005Metric_Pad0.72x0.64mm_HandSolder
- removed R174, R175, R176, R177, R178, R179, R181, R182, R185, R186, R187, R188, R189, R190, R196, R197, R198, R199, R200, R201, R202, R203, R209, R210, R211, R212, R213, R214, R215, R216, R222, R223, R224, R225, R226, R227, R228, R229, R235, R236, R237, R238, R239, R240, R241, R242, R248, R249, R250, R251, R252, R253, R254, R255, R261, R262, R263, R264, R265, R266, R267, R268, R274, R275: 4.7K, Resistor_SMD:R_0402_1005Metric
- removed R180, R195, R208, R221, R234, R247, R260, R273: R-1k-0402, cm5-module-Library:R_0402_1005Metric
- added C100: M1, Capacitor_SMD:C_0402_1005Metric, F.Cu at (380.2, 155.0)
- added C101: 12P, Capacitor_SMD:C_0402_1005Metric, F.Cu at (380.2, 157.0)
- added C102: M1, Capacitor_SMD:C_0402_1005Metric, F.Cu at (383.0, 149.1)
- added C103: M1, Capacitor_SMD:C_0402_1005Metric, F.Cu at (383.0, 151.1)
- added C104: 1M, Capacitor_SMD:C_0402_1005Metric, F.Cu at (383.0, 153.0)
- added C188: 12P, Capacitor_SMD:C_0402_1005Metric, F.Cu at (383.0, 155.0)
- added C189: 1M, Capacitor_SMD:C_0603_1608Metric, F.Cu at (376.7, 151.9)
- added C190: 470P, Capacitor_SMD:C_0402_1005Metric, F.Cu at (383.0, 157.0)
- added C191: M1, Capacitor_SMD:C_0402_1005Metric, F.Cu at (397.0, 178.3)
- added C192: M1, Capacitor_SMD:C_0402_1005Metric, F.Cu at (341.1, 182.6)
- added C193: 1N, Capacitor_SMD:C_0603_1608Metric, F.Cu at (397.5, 173.6)
- added C194: 1N, Capacitor_SMD:C_0603_1608Metric, F.Cu at (341.6, 177.8)
- added C196: 100n, Capacitor_SMD:C_0402_1005Metric, B.Cu at (179.5, 189.6)
- added C197: 22u, Capacitor_SMD:C_0603_1608Metric_Pad1.08x0.95mm_HandSolder, B.Cu at (175.5, 188.9)
- added C198: 22u, Capacitor_SMD:C_0603_1608Metric_Pad1.08x0.95mm_HandSolder, B.Cu at (175.5, 192.5)
- added C199: 100n, Capacitor_SMD:C_0402_1005Metric, B.Cu at (164.8, 189.1)
- added C200: 100n, Capacitor_SMD:C_0402_1005Metric, B.Cu at (166.1, 190.4)
- added C201: 22u, Capacitor_SMD:C_0603_1608Metric_Pad1.08x0.95mm_HandSolder, B.Cu at (175.4, 196.0)
- added C202: 100n, Capacitor_SMD:C_0402_1005Metric, B.Cu at (163.5, 191.0)
- added C203: 22u, Capacitor_SMD:C_0603_1608Metric_Pad1.08x0.95mm_HandSolder, B.Cu at (181.2, 189.6)
- added C204: 22u, Capacitor_SMD:C_0603_1608Metric_Pad1.08x0.95mm_HandSolder, B.Cu at (181.2, 239.1)
- added C205: 100n, Capacitor_SMD:C_0402_1005Metric, B.Cu at (179.5, 239.1)
- added C206: 22u, Capacitor_SMD:C_0603_1608Metric_Pad1.08x0.95mm_HandSolder, B.Cu at (175.5, 238.4)
- added C207: 22u, Capacitor_SMD:C_0603_1608Metric_Pad1.08x0.95mm_HandSolder, B.Cu at (175.5, 242.0)
- added C208: 22u, Capacitor_SMD:C_0603_1608Metric_Pad1.08x0.95mm_HandSolder, B.Cu at (175.4, 245.5)
- added C209: 100n, Capacitor_SMD:C_0402_1005Metric, B.Cu at (164.8, 238.6)
- added C210: 100n, Capacitor_SMD:C_0402_1005Metric, B.Cu at (166.1, 239.8)
- added C211: 100n, Capacitor_SMD:C_0402_1005Metric, B.Cu at (163.5, 240.5)
- added C212: 22u, Capacitor_SMD:C_0603_1608Metric_Pad1.08x0.95mm_HandSolder, B.Cu at (181.2, 164.9)
- added C213: 100n, Capacitor_SMD:C_0402_1005Metric, B.Cu at (179.5, 164.9)
- added C214: 22u, Capacitor_SMD:C_0603_1608Metric_Pad1.08x0.95mm_HandSolder, B.Cu at (175.5, 164.2)
- added C215: 22u, Capacitor_SMD:C_0603_1608Metric_Pad1.08x0.95mm_HandSolder, B.Cu at (175.5, 167.8)
- added C216: 22u, Capacitor_SMD:C_0603_1608Metric_Pad1.08x0.95mm_HandSolder, B.Cu at (175.4, 171.3)
- added C217: 100n, Capacitor_SMD:C_0402_1005Metric, B.Cu at (164.8, 164.4)
- added C218: 100n, Capacitor_SMD:C_0402_1005Metric, B.Cu at (166.1, 165.6)
- added C219: 100n, Capacitor_SMD:C_0402_1005Metric, B.Cu at (163.5, 166.3)
- added C220: 22u, Capacitor_SMD:C_0603_1608Metric_Pad1.08x0.95mm_HandSolder, B.Cu at (181.2, 214.4)
- added C221: 100n, Capacitor_SMD:C_0402_1005Metric, B.Cu at (179.5, 214.4)
- added C222: 22u, Capacitor_SMD:C_0603_1608Metric_Pad1.08x0.95mm_HandSolder, B.Cu at (175.5, 213.7)
- added C223: 22u, Capacitor_SMD:C_0603_1608Metric_Pad1.08x0.95mm_HandSolder, B.Cu at (175.5, 217.2)
- added C224: 22u, Capacitor_SMD:C_0603_1608Metric_Pad1.08x0.95mm_HandSolder, B.Cu at (175.4, 220.8)
- added C225: 100n, Capacitor_SMD:C_0402_1005Metric, B.Cu at (164.8, 213.8)
- added C226: 100n, Capacitor_SMD:C_0402_1005Metric, B.Cu at (166.1, 215.1)
- added C227: 100n, Capacitor_SMD:C_0402_1005Metric, B.Cu at (163.5, 215.8)
- added C281: M1, Capacitor_SMD:C_0402_1005Metric, F.Cu at (397.8, 163.7)
- added C282: 10M, Capacitor_SMD:C_0603_1608Metric, F.Cu at (397.7, 168.5)
- added C283: 10M, Capacitor_SMD:C_0603_1608Metric, F.Cu at (366.7, 163.3)
- added C284: 10M, Capacitor_SMD:C_0805_2012Metric, F.Cu at (393.5, 168.8)
- added C285: 10M, Capacitor_SMD:C_0603_1608Metric, F.Cu at (366.7, 165.8)
- added C286: 10M, Capacitor_SMD:C_0603_1608Metric, F.Cu at (366.7, 168.3)
- added C57: M1, Capacitor_SMD:C_0402_1005Metric, F.Cu at (353.5, 149.8)
- added C58: M1, Capacitor_SMD:C_0402_1005Metric, F.Cu at (353.5, 151.8)
- added C59: M1, Capacitor_SMD:C_0402_1005Metric, F.Cu at (353.5, 153.8)
- added C60: M1, Capacitor_SMD:C_0402_1005Metric, F.Cu at (353.5, 155.7)
- added C61: M1, Capacitor_SMD:C_0402_1005Metric, F.Cu at (353.5, 157.7)
- added C62: M1, Capacitor_SMD:C_0402_1005Metric, F.Cu at (353.5, 159.7)
- added C63: M1, Capacitor_SMD:C_0402_1005Metric, F.Cu at (353.5, 161.6)
- added C64: M1, Capacitor_SMD:C_0402_1005Metric, F.Cu at (356.4, 149.8)
- added C65: M1, Capacitor_SMD:C_0402_1005Metric, F.Cu at (356.4, 151.8)
- added C81: M1, Capacitor_SMD:C_0402_1005Metric, F.Cu at (356.4, 153.8)
- added C82: M1, Capacitor_SMD:C_0402_1005Metric, F.Cu at (356.4, 155.7)
- added C83: 1M, Capacitor_SMD:C_0603_1608Metric, F.Cu at (362.7, 163.3)
- added C84: 12P, Capacitor_SMD:C_0402_1005Metric, F.Cu at (356.4, 157.7)
- added C85: 12P, Capacitor_SMD:C_0402_1005Metric, F.Cu at (356.4, 159.7)
- added C86: M1, Capacitor_SMD:C_0402_1005Metric, F.Cu at (356.4, 161.6)
- added C87: M1, Capacitor_SMD:C_0402_1005Metric, F.Cu at (359.3, 149.8)
- added C88: 1M, Capacitor_SMD:C_0603_1608Metric, F.Cu at (362.7, 165.8)
- added C89: M1, Capacitor_SMD:C_0402_1005Metric, F.Cu at (359.3, 151.8)
- added C90: 1M, Capacitor_SMD:C_0603_1608Metric, F.Cu at (362.7, 168.3)
- added C91: 1M, Capacitor_SMD:C_0603_1608Metric, F.Cu at (362.7, 170.8)
- added C92: 1M, Capacitor_SMD:C_0603_1608Metric, F.Cu at (362.7, 173.3)
- added C93: 1P5, Capacitor_SMD:C_0402_1005Metric, F.Cu at (359.3, 153.8)
- added C94: 1P5, Capacitor_SMD:C_0402_1005Metric, F.Cu at (359.3, 155.7)
- added C95: 1N, Capacitor_SMD:C_1206_3216Metric, F.Cu at (387.3, 156.1)
- added C96: M1, Capacitor_SMD:C_0402_1005Metric, F.Cu at (380.2, 149.1)
- added C97: M1, Capacitor_SMD:C_0402_1005Metric, F.Cu at (380.2, 151.1)
- added C98: 10M, Capacitor_SMD:C_0603_1608Metric, F.Cu at (376.7, 149.4)
- added C99: M1, Capacitor_SMD:C_0402_1005Metric, F.Cu at (380.2, 153.0)
- added D13: LED, LED_SMD:LED_0603_1608Metric, F.Cu at (337.4, 166.2)
- added D14: LED, LED_SMD:LED_0603_1608Metric, F.Cu at (337.4, 168.8)
- added D20: LED, LED_SMD:LED_0603_1608Metric, F.Cu at (337.4, 171.4)
- added D21: 1N5819WS, Diode_SMD:D_SOD-323, F.Cu at (341.6, 166.4)
- added D22: PUSB3F96X, cm5-module-Library:SOT1176-1, B.Cu at (64.1, 135.8)
- added D23: PUSB3F96X, cm5-module-Library:SOT1176-1, B.Cu at (64.1, 138.9)
- added D24: 1N5819WS, Diode_SMD:D_SOD-323, F.Cu at (341.6, 169.3)
- added D25: SMAJ24A, Diode_SMD:D_SMA, F.Cu at (383.1, 164.9)
- added D26: DNP, Diode_SMD:D_SOD-323, F.Cu at (393.4, 173.8)
- added D27: DNP, Diode_SMD:D_SOD-323, F.Cu at (337.5, 178.0)
- added D36: DNP, Diode_SMD:D_SOD-323, F.Cu at (393.4, 176.7)
- added D37: DNP, Diode_SMD:D_SOD-323, F.Cu at (337.5, 181.0)
- added D42: DNP, Diode_SMD:D_SOD-323, F.Cu at (376.9, 164.1)
- added D43: DNP, Diode_SMD:D_SOD-323, F.Cu at (376.9, 167.1)
- added D44: DNP, Diode_SMD:D_SOD-323, F.Cu at (376.9, 170.0)
- added D45: DNP, Diode_SMD:D_SOD-323, F.Cu at (376.9, 173.0)
- added F1: SMD1812P150TF/24, Fuse:Fuse_1812_4532Metric_Pad1.30x3.40mm_HandSolder, F.Cu at (385.6, 169.7)
- added FB1: GZ1608D601TF, Inductor_SMD:L_0603_1608Metric, F.Cu at (376.7, 154.4)
- added FB2: GZ1608D601TF, Inductor_SMD:L_0603_1608Metric, F.Cu at (376.7, 156.9)
- added FB3: GZ1608D601TF, Inductor_SMD:L_0603_1608Metric, F.Cu at (376.7, 159.4)
- added FB4: GZ1608D601TF, Inductor_SMD:L_0603_1608Metric, F.Cu at (366.7, 170.8)
- added FB5: GZ1608D601TF, Inductor_SMD:L_0603_1608Metric, F.Cu at (366.7, 173.3)
- added FB6: GZ1608D601TF, Inductor_SMD:L_0603_1608Metric, F.Cu at (370.7, 163.3)
- added FL1: ACM2012-900-2P-T002, Inductor_SMD:L_CommonModeChoke_Coilcraft_0805USB, F.Cu at (383.4, 174.2)
- added J40: Micro_SD_Card, Connector_Card:microSD_HC_Molex_47219-2001, F.Cu at (343.7, 156.9)
- added J41: RJHSE5383, Connector_RJ:RJ45_Amphenol_RJHSE538X, F.Cu at (381.5, 139.3)
- added J42: USB_C_Receptacle_USB2.0, Connector_USB:USB_C_Receptacle_GCT_USB4105-xx-A_16P_TopMnt_Horizontal, F.Cu at (361.2, 185.7)
- added J43: ATX-24, Connector_Molex:Molex_Mini-Fit_Jr_5566-24A_2x12_P4.20mm_Vertical, F.Cu at (198.5, 108.1)
- added L25: 1uH, Inductor_SMD:L_0603_1608Metric_Pad1.05x0.95mm_HandSolder, B.Cu at (177.1, 188.9)
- added L26: 1uH, Inductor_SMD:L_0603_1608Metric_Pad1.05x0.95mm_HandSolder, B.Cu at (177.1, 192.5)
- added L27: 1uH, Inductor_SMD:L_0603_1608Metric_Pad1.05x0.95mm_HandSolder, B.Cu at (177.2, 196.0)
- added L28: 1uH, Inductor_SMD:L_0603_1608Metric_Pad1.05x0.95mm_HandSolder, B.Cu at (177.1, 238.4)
- added L29: 1uH, Inductor_SMD:L_0603_1608Metric_Pad1.05x0.95mm_HandSolder, B.Cu at (177.1, 242.0)
- added L30: 1uH, Inductor_SMD:L_0603_1608Metric_Pad1.05x0.95mm_HandSolder, B.Cu at (177.2, 245.5)
- added L31: 1uH, Inductor_SMD:L_0603_1608Metric_Pad1.05x0.95mm_HandSolder, B.Cu at (177.1, 164.2)
- added L32: 1uH, Inductor_SMD:L_0603_1608Metric_Pad1.05x0.95mm_HandSolder, B.Cu at (177.1, 167.8)
- added L33: 1uH, Inductor_SMD:L_0603_1608Metric_Pad1.05x0.95mm_HandSolder, B.Cu at (177.2, 171.3)
- added L34: 1uH, Inductor_SMD:L_0603_1608Metric_Pad1.05x0.95mm_HandSolder, B.Cu at (177.1, 213.7)
- added L35: 1uH, Inductor_SMD:L_0603_1608Metric_Pad1.05x0.95mm_HandSolder, B.Cu at (177.1, 217.3)
- added L36: 1uH, Inductor_SMD:L_0603_1608Metric_Pad1.05x0.95mm_HandSolder, B.Cu at (177.2, 220.8)
- added R100: 100R, Capacitor_SMD:C_0603_1608Metric, F.Cu at (370.7, 165.8)
- added R101: 10K, Resistor_SMD:R_0402_1005Metric, F.Cu at (355.3, 133.3)
- added R102: 0R, Capacitor_SMD:C_0603_1608Metric, F.Cu at (370.7, 168.3)
- added R103: 1M, Resistor_SMD:R_1206_3216Metric, F.Cu at (394.0, 149.8)
- added R105: 49R9, Resistor_SMD:R_0402_1005Metric, F.Cu at (396.8, 131.3)
- added R106: 49R9, Resistor_SMD:R_0402_1005Metric, F.Cu at (396.8, 133.3)
- added R107: 49R9, Resistor_SMD:R_0402_1005Metric, F.Cu at (396.8, 135.3)
- added R108: 330R, Resistor_SMD:R_0402_1005Metric, F.Cu at (396.8, 137.3)
- added R111: 330R, Resistor_SMD:R_0402_1005Metric, F.Cu at (396.8, 139.3)
- added R112: 49R9, Resistor_SMD:R_0402_1005Metric, F.Cu at (396.8, 141.3)
- added R113: 10K, Resistor_SMD:R_0402_1005Metric, F.Cu at (396.8, 143.3)
- added R114: 10K, Resistor_SMD:R_0402_1005Metric, F.Cu at (399.7, 131.3)
- added R115: 12K1, Resistor_SMD:R_0402_1005Metric, F.Cu at (399.7, 133.3)
- added R116: 10K, Resistor_SMD:R_0402_1005Metric, F.Cu at (399.7, 135.3)
- added R117: 10K, Resistor_SMD:R_0402_1005Metric, F.Cu at (399.7, 137.3)
- added R118: 10K, Resistor_SMD:R_0402_1005Metric, F.Cu at (399.7, 139.3)
- added R119: 10K, Resistor_SMD:R_0402_1005Metric, F.Cu at (399.7, 141.3)
- added R120: 10K, Resistor_SMD:R_0402_1005Metric, F.Cu at (399.7, 143.3)
- added R121: 10K, Resistor_SMD:R_0402_1005Metric, F.Cu at (402.6, 131.3)
- added R122: 33R, Resistor_SMD:R_0402_1005Metric, F.Cu at (402.6, 133.3)
- added R123: 33R, Resistor_SMD:R_0402_1005Metric, F.Cu at (402.6, 135.3)
- added R124: 33R, Resistor_SMD:R_0402_1005Metric, F.Cu at (402.6, 137.3)
- added R125: 75R, Capacitor_SMD:C_0603_1608Metric, F.Cu at (397.5, 176.1)
- added R126: 75R, Capacitor_SMD:C_0603_1608Metric, F.Cu at (341.6, 180.3)
- added R127: R-2k2-0402, Resistor_SMD:R_0402_1005Metric_Pad0.72x0.64mm_HandSolder, F.Cu at (59.0, 106.6)
- added R276: 330R, Resistor_SMD:R_0402_1005Metric, F.Cu at (355.3, 135.3)
- added R277: 330R, Resistor_SMD:R_0402_1005Metric, F.Cu at (355.3, 137.3)
- added R278: 330R, Resistor_SMD:R_0402_1005Metric, F.Cu at (355.3, 139.3)
- added R279: 10K, Resistor_SMD:R_0402_1005Metric, F.Cu at (355.3, 141.3)
- added R280: 10K, Resistor_SMD:R_0402_1005Metric, F.Cu at (355.3, 143.3)
- added R281: 10K, Resistor_SMD:R_0402_1005Metric, F.Cu at (355.3, 145.2)
- added R282: 10K, Resistor_SMD:R_0402_1005Metric, F.Cu at (355.3, 147.2)
- added R283: 33R, Resistor_SMD:R_0402_1005Metric, F.Cu at (358.2, 131.3)
- added R284: 33R, Resistor_SMD:R_0402_1005Metric, F.Cu at (358.2, 133.3)
- added R285: 33R, Resistor_SMD:R_0402_1005Metric, F.Cu at (358.2, 135.3)
- added R286: 33R, Resistor_SMD:R_0402_1005Metric, F.Cu at (358.2, 137.3)
- added R287: 33R, Resistor_SMD:R_0402_1005Metric, F.Cu at (358.2, 139.3)
- added R288: 33R, Resistor_SMD:R_0402_1005Metric, F.Cu at (358.2, 141.3)
- added R289: 33R, Resistor_SMD:R_0402_1005Metric, F.Cu at (358.2, 143.3)
- added R290: 33R, Resistor_SMD:R_0402_1005Metric, F.Cu at (358.2, 145.2)
- added R291: 33R, Resistor_SMD:R_0402_1005Metric, F.Cu at (358.2, 147.2)
- added R292: 33R, Resistor_SMD:R_0402_1005Metric, F.Cu at (361.1, 131.3)
- added R293: 33R, Resistor_SMD:R_0402_1005Metric, F.Cu at (361.1, 133.3)
- added R294: 33R, Resistor_SMD:R_0402_1005Metric, F.Cu at (361.1, 135.3)
- added R295: 33R, Resistor_SMD:R_0402_1005Metric, F.Cu at (361.1, 137.3)
- added R296: 33R, Resistor_SMD:R_0402_1005Metric, F.Cu at (361.1, 139.3)
- added R297: 33R, Resistor_SMD:R_0402_1005Metric, F.Cu at (361.1, 141.3)
- added R298: 33R, Resistor_SMD:R_0402_1005Metric, F.Cu at (361.1, 143.3)
- added R299: 33R, Resistor_SMD:R_0402_1005Metric, F.Cu at (361.1, 145.2)
- added R300: 33R, Resistor_SMD:R_0402_1005Metric, F.Cu at (361.1, 147.2)
- added R301: 33R, Resistor_SMD:R_0402_1005Metric, F.Cu at (364.0, 131.3)
- added R302: 33R, Resistor_SMD:R_0402_1005Metric, F.Cu at (364.0, 133.3)
- added R303: 33R, Resistor_SMD:R_0402_1005Metric, F.Cu at (364.0, 135.3)
- added R304: 33R, Resistor_SMD:R_0402_1005Metric, F.Cu at (364.0, 137.3)
- added R305: 33R, Resistor_SMD:R_0402_1005Metric, F.Cu at (364.0, 139.3)
- added R306: 33R, Resistor_SMD:R_0402_1005Metric, F.Cu at (364.0, 141.3)
- added R307: 33R, Resistor_SMD:R_0402_1005Metric, F.Cu at (364.0, 143.3)
- added R308: 33R, Resistor_SMD:R_0402_1005Metric, F.Cu at (364.0, 145.2)
- added R309: 33R, Resistor_SMD:R_0402_1005Metric, F.Cu at (364.0, 147.2)
- added R310: 33R, Resistor_SMD:R_0402_1005Metric, F.Cu at (366.9, 131.3)
- added R311: 33R, Resistor_SMD:R_0402_1005Metric, F.Cu at (366.9, 133.3)
- added R312: 33R, Resistor_SMD:R_0402_1005Metric, F.Cu at (366.9, 135.3)
- added R313: 33R, Resistor_SMD:R_0402_1005Metric, F.Cu at (366.9, 137.3)
- added R314: 33R, Resistor_SMD:R_0402_1005Metric, F.Cu at (366.9, 139.3)
- added R315: 33R, Resistor_SMD:R_0402_1005Metric, F.Cu at (366.9, 141.3)
- added R316: 33R, Resistor_SMD:R_0402_1005Metric, F.Cu at (366.9, 143.3)
- added R317: 33R, Resistor_SMD:R_0402_1005Metric, F.Cu at (366.9, 145.2)
- added R318: 33R, Resistor_SMD:R_0402_1005Metric, F.Cu at (366.9, 147.2)
- added R319: 33R, Resistor_SMD:R_0402_1005Metric, F.Cu at (369.9, 131.3)
- added R320: 33R, Resistor_SMD:R_0402_1005Metric, F.Cu at (369.9, 133.3)
- added R321: 33R, Resistor_SMD:R_0402_1005Metric, F.Cu at (369.9, 135.3)
- added R322: 33R, Resistor_SMD:R_0402_1005Metric, F.Cu at (369.9, 137.3)
- added R323: 10K, Resistor_SMD:R_0402_1005Metric, F.Cu at (369.9, 139.3)
- added R324: 10K, Resistor_SMD:R_0402_1005Metric, F.Cu at (369.9, 141.3)
- added R325: 33R, Resistor_SMD:R_0402_1005Metric, F.Cu at (380.5, 168.2)
- added R326: 33R, Resistor_SMD:R_0402_1005Metric, F.Cu at (380.5, 170.2)
- added R327: 33R, Resistor_SMD:R_0402_1005Metric, F.Cu at (380.5, 172.2)
- added R328: 33R, Resistor_SMD:R_0402_1005Metric, F.Cu at (380.5, 174.2)
- added R329: 4.7K, Resistor_SMD:R_0402_1005Metric, B.Cu at (173.2, 187.3)
- added R330: 4.7K, Resistor_SMD:R_0402_1005Metric, B.Cu at (173.2, 184.5)
- added R331: 4.7K, Resistor_SMD:R_0402_1005Metric, B.Cu at (173.2, 192.9)
- added R332: 4.7K, Resistor_SMD:R_0402_1005Metric, B.Cu at (173.2, 194.3)
- added R333: 4.7K, Resistor_SMD:R_0402_1005Metric, B.Cu at (173.2, 188.7)
- added R334: 4.7K, Resistor_SMD:R_0402_1005Metric, B.Cu at (173.2, 190.1)
- added R335: 4.7K, Resistor_SMD:R_0402_1005Metric, B.Cu at (173.2, 191.5)
- added R336: 4.7K, Resistor_SMD:R_0402_1005Metric, B.Cu at (173.2, 185.9)
- added R337: 4.7K, Resistor_SMD:R_0402_1005Metric, B.Cu at (173.2, 243.8)
- added R338: 4.7K, Resistor_SMD:R_0402_1005Metric, B.Cu at (173.2, 239.6)
- added R339: 4.7K, Resistor_SMD:R_0402_1005Metric, B.Cu at (173.2, 241.0)
- added R340: 4.7K, Resistor_SMD:R_0402_1005Metric, B.Cu at (173.2, 242.4)
- added R341: 4.7K, Resistor_SMD:R_0402_1005Metric, B.Cu at (173.2, 234.0)
- added R342: 4.7K, Resistor_SMD:R_0402_1005Metric, B.Cu at (173.2, 236.8)
- added R343: 4.7K, Resistor_SMD:R_0402_1005Metric, B.Cu at (173.2, 238.2)
- added R344: 4.7K, Resistor_SMD:R_0402_1005Metric, B.Cu at (173.2, 235.4)
- added R345: 4.7K, Resistor_SMD:R_0402_1005Metric, B.Cu at (173.2, 169.6)
- added R346: 4.7K, Resistor_SMD:R_0402_1005Metric, B.Cu at (173.2, 165.4)
- added R347: 4.7K, Resistor_SMD:R_0402_1005Metric, B.Cu at (173.2, 166.8)
- added R348: 4.7K, Resistor_SMD:R_0402_1005Metric, B.Cu at (173.2, 168.2)
- added R349: 4.7K, Resistor_SMD:R_0402_1005Metric, B.Cu at (173.2, 159.7)
- added R350: 4.7K, Resistor_SMD:R_0402_1005Metric, B.Cu at (173.2, 162.6)
- added R351: 4.7K, Resistor_SMD:R_0402_1005Metric, B.Cu at (173.2, 164.0)
- added R352: 4.7K, Resistor_SMD:R_0402_1005Metric, B.Cu at (173.2, 161.1)
- added R353: 4.7K, Resistor_SMD:R_0402_1005Metric, B.Cu at (173.2, 219.1)
- added R354: 4.7K, Resistor_SMD:R_0402_1005Metric, B.Cu at (173.2, 214.8)
- added R355: 4.7K, Resistor_SMD:R_0402_1005Metric, B.Cu at (173.2, 216.2)
- added R356: 4.7K, Resistor_SMD:R_0402_1005Metric, B.Cu at (173.2, 217.6)
- added R357: 4.7K, Resistor_SMD:R_0402_1005Metric, B.Cu at (173.2, 209.2)
- added R358: 4.7K, Resistor_SMD:R_0402_1005Metric, B.Cu at (173.2, 212.0)
- added R359: 4.7K, Resistor_SMD:R_0402_1005Metric, B.Cu at (173.2, 213.4)
- added R360: 4.7K, Resistor_SMD:R_0402_1005Metric, B.Cu at (173.2, 210.6)
- added R99: 100R, Resistor_SMD:R_0402_1005Metric, F.Cu at (355.3, 131.3)
- added U10: W25x_SOIC8 (DNP), Package_SO:SOIC-8_3.9x4.9mm_P1.27mm, F.Cu at (356.3, 166.0)
- added U11: W25x_WSOIC8 (DNP), Package_SO:SOIC-8_3.9x4.9mm_P1.27mm, F.Cu at (356.3, 174.0)
- added U13: LAN8720A, Package_DFN_QFN:VQFN-24-1EP_4x4mm_P0.5mm_EP2.5x2.5mm_ThermalVias, F.Cu at (388.0, 151.3)
- added U14: QSFP_Conn, memblaze2qmtech:QSFP_Conn_w_Cage, F.Cu at (173.2, 197.7)
- added U15: SN74LV595APWR, Package_SO:TSSOP-16_4.4x5mm_P0.65mm, F.Cu at (365.5, 152.1)
- added U16: SN74LV595APWR, Package_SO:TSSOP-16_4.4x5mm_P0.65mm, F.Cu at (365.5, 158.7)
- added U17: QSFP_Conn, memblaze2qmtech:QSFP_Conn_w_Cage, F.Cu at (173.2, 247.2)
- added U18: QSFP_Conn, memblaze2qmtech:QSFP_Conn_w_Cage, F.Cu at (173.2, 173.0)
- added U19: QSFP_Conn, memblaze2qmtech:QSFP_Conn_w_Cage, F.Cu at (173.2, 222.5)
- added U30: AP63200WU, Package_TO_SOT_SMD:TSOT-23-6, F.Cu at (393.8, 165.1)
- added U8: TL431DBZ, Resistor_SMD:R_0402_1005Metric, F.Cu at (369.9, 143.3)
- added U9: STM32H563VGT6, Package_QFP:LQFP-100_14x14mm_P0.5mm, F.Cu at (344.6, 139.6)
- added Y1: X322525MOB4SI, Crystal:Crystal_SMD_3225-4Pin_3.2x2.5mm, F.Cu at (393.8, 153.7)
- added Y2: X322525MOB4SI, Crystal:Crystal_SMD_3225-4Pin_3.2x2.5mm, F.Cu at (346.3, 167.2)
- BT1, C167, C21, C22, C23, C24, C25, C26, C27, C28, C29, C30, C31, C32, C33, C34, C35, C36, C37, C38, C41, C42, C43, C44, C45, C46, C47, C48, C49, C5, C50, C51, C52, C53, C55, C56, C6, C71, C72, C74, C75, C78, C9, D10, D9, J10, L2, L3, L4, R109: moved to B.Cu
- moved R93 294.2 mm to (184.5, 45.8), turned to -90 degrees
- moved R94 292.8 mm to (182.3, 45.9), turned to 90 degrees
- moved C69 291.4 mm to (179.6, 46.0), turned to 180 degrees
- moved C70 279.9 mm to (170.5, 46.2)
- moved C68 279.8 mm to (172.3, 50.0), turned to 90 degrees
- moved U6 276.4 mm to (176.4, 49.9)
- moved R92 274.1 mm to (176.0, 53.6)
- moved L5 273.1 mm to (167.1, 47.6), turned to 90 degrees
- moved R90 268.1 mm to (162.7, 46.4)
- moved C67 267.9 mm to (170.0, 50.0), turned to 90 degrees
- moved D1 234.5 mm to (173.6, 115.9), turned to 0 degrees
- moved D2 232.7 mm to (173.6, 114.2), turned to 0 degrees
- moved R1 232.6 mm to (170.8, 115.9), turned to 0 degrees
- moved R2 231.1 mm to (170.8, 114.3), turned to 0 degrees
- moved R4 200.6 mm to (127.3, 79.8), turned to 180 degrees
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Connections:
- net /REFCLKO1+ renamed /REFCLKO1.+
- net /REFCLKO1- renamed /REFCLKO1.-
- net /REFCLKO2+ renamed /REFCLKO2.+
- net /REFCLKO2- renamed /REFCLKO2.-
- net Net-(C7-Pad1) renamed /RPiUSB2_VBUS
- net Net-(U2-REFCLKIN) renamed /PCIe.REFCLK_PIN-
- net Net-(U2-REFCLKIP) renamed /PCIe.REFCLK_PIN+
- net Net-(U2-REFCLKN[0]) renamed /REFCLK1_PIN+
- net Net-(U2-REFCLKN[1]) renamed /REFCLK2_PIN+
- net Net-(U2-REFCLKON[1]) renamed /REFCLKO1_PIN-
- net Net-(U2-REFCLKON[2]) renamed /REFCLKO2_PIN-
- net Net-(U2-REFCLKON[3]) renamed /REFCLKO3_PIN-
- net Net-(U2-REFCLKON[4]) renamed /REFCLKO4_PIN-
- net Net-(U2-REFCLKON[5]) renamed /REFCLKO5_PIN-
- net Net-(U2-REFCLKON[7]) renamed /REFCLKO7_PIN-
- net Net-(U2-REFCLKOP[1]) renamed /REFCLKO1_PIN+
- net Net-(U2-REFCLKOP[2]) renamed /REFCLKO2_PIN+
- net Net-(U2-REFCLKOP[3]) renamed /REFCLKO3_PIN+
- net Net-(U2-REFCLKOP[4]) renamed /REFCLKO4_PIN+
- net Net-(U2-REFCLKOP[5]) renamed /REFCLKO5_PIN+
- net Net-(U2-REFCLKOP[7]) renamed /REFCLKO7_PIN+
- net Net-(U2-REFCLKP[0]) renamed /REFCLK1_PIN-
- net Net-(U2-REFCLKP[1]) renamed /REFCLK2_PIN-
- net Net-(U5-VCC) renamed /RPiUART_VBUS
- J10 pad 9: GND -> (no net)
- J10 pad SH1: (no net) -> GND
- J10 pad SH2: (no net) -> GND
- J10 pad SH3: (no net) -> GND
- J10 pad SH4: (no net) -> GND
- J22 pad A16: /FPGA0_TX.+ -> /FPGA2_TX.+
- J22 pad A17: /FPGA0_TX.- -> /FPGA2_TX.-
- J22 pad B14: /FPGA0_RX.+ -> /FPGA2_RX.+
- J22 pad B15: /FPGA0_RX.- -> /FPGA2_RX.-
- J37 pad A16: /FPGA1_TX.+ -> /FPGA3_TX.+
- J37 pad A17: /FPGA1_TX.- -> /FPGA3_TX.-
- J37 pad B14: /FPGA1_RX.+ -> /FPGA3_RX.+
- J37 pad B15: /FPGA1_RX.- -> /FPGA3_RX.-
- R60 pad 2: /REFCLKO3+ -> /REFCLKO3.+
- R61 pad 2: /REFCLKO3- -> /REFCLKO3.-
- R62 pad 2: /REFCLKO4+ -> /REFCLKO4.+
- R63 pad 2: /REFCLKO4- -> /REFCLKO4.-
- R64 pad 2: /REFCLKO5+ -> /REFCLKO5.+
- R65 pad 2: /REFCLKO5- -> /REFCLKO5.-
- R66 pad 2: /REFCLKO7+ -> /REFCLKO7.+
- R67 pad 2: /REFCLKO7- -> /REFCLKO7.-
- R72 pad 1: /REFCLKO3+ -> /REFCLKO3.+
- R73 pad 1: /REFCLKO3- -> /REFCLKO3.-
- R74 pad 1: /REFCLKO4+ -> /REFCLKO4.+
- R75 pad 1: /REFCLKO4- -> /REFCLKO4.-
- R76 pad 1: /REFCLKO5+ -> /REFCLKO5.+
- R77 pad 1: /REFCLKO5- -> /REFCLKO5.-
- R78 pad 1: /REFCLKO7+ -> /REFCLKO7.+
- R79 pad 1: /REFCLKO7- -> /REFCLKO7.-
- U1 pad 3: unconnected-(U1-~{FLG}-Pad3) -> Net-(U1-~{FLG})
Routing:
- net GND: track 0.00 -> 235.9 mm, vias 0 -> 291
- net /FPGA1_RX.+: track 0.00 -> 117.1 mm, vias 0 -> 2
- net /FPGA1_RX.-: track 0.00 -> 116.8 mm, vias 0 -> 2
- net /FPGA1_TX.+: track 0.00 -> 108.9 mm, vias 0 -> 2
- net /FPGA1_TX.-: track 0.00 -> 108.5 mm, vias 0 -> 2
- net +3V3: track 0.00 -> 107.5 mm, vias 0 -> 59
- net /GPIO5: track 0.00 -> 97.3 mm, vias 0 -> 2
- net /GPIO4: track 0.00 -> 96.0 mm, vias 0 -> 2
- net /CC2: track 0.00 -> 90.0 mm, vias 0 -> 2
- net /CC1: track 0.00 -> 89.4 mm, vias 0 -> 4
- net /USB.D+: track 0.00 -> 85.8 mm, vias 0 -> 4
- net /USB.D-: track 0.00 -> 85.8 mm, vias 0 -> 2
- net /ETH.D4+: track 0.00 -> 82.5 mm, vias 0 -> 1
- net /ETH.D3-: track 0.00 -> 81.7 mm, vias 0 -> 2
- net /ETH.D4-: track 0.00 -> 81.6 mm, vias 0 -> 1
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- added copper zone on In1.Cu, net GND
- added copper zone on In2.Cu, net GND
- added copper zone on F.Cu, net Net-(C70-Pad1)
Other:
- outline, holes or cut-outs redrawn
- board text added: "D6"
- board text added: "D7"
- board text added: "D8"
- board text added: "FPGA0"
- board text added: "FPGA1"
- board text added: "FPGA2"
- board text added: "FPGA3"
- board text added: "VBUS"
