File: 1-baseboard/TentaLab/tentalab.kicad_pcb (KiCad board)
At the start: 4 copper layers, 171.4 x 243.8 mm, 507 parts, among them J1 USB-A_USB-303WSD-BRY, J10 Micro_SD_Card, J11 RPI_HEADER, J12 RPI_OPTIONS, J13 RJ45_HC612601A-M893-A, J14 PCIe, J15 PCIe, J16 12V ATX, J17 JTAG_0, J18 JTAG_0, J19 JTAG_0, J2 JTAG_UPSTREAM, J20 Jack-DC, J21 FPGA_RST_nPRSNT, J22 PCIe, J23 RPi UART, J24 JTAG_0, J25 JTAG_SKIP_0, J26 JTAG_SKIP_0, J27 JTAG_SKIP_0, J28 JTAG_SKIP_0, J29 Conn_01x22_Female, J3 CM5_1-100_3mm-stack, J30 Conn_01x22_Female, J37 PCIe, J4 CM5_101-200_3mm-stack, J40 Micro_SD_Card, J41 RJHSE5383, J42 USB_C_Receptacle_USB2.0, J43 ATX-24, J5 HDMI_A, J6 Conn_Coaxial_Small, J7 HDMI_A, J8 Conn_01x04, J9 RPi USB2, SW1 PWR_BTN, U1 AP22615AWU-7, U10 W25x_SOIC8 (DNP), U11 W25x_WSOIC8 (DNP), U12 RT9742SNGV, U13 LAN8720A, U14 QSFP_Conn, U15 SN74LV595APWR, U16 SN74LV595APWR, U17 QSFP_Conn, U18 QSFP_Conn, U19 QSFP_Conn, U2 PI7C9X2G608ELBZXAE, U3 TPS62821DLC, U30 AP63200WU, U4 M93C86, U5 CH330N, U6 TPS563200, U7 AP22615AWU-7, U8 TL431DBZ, U9 STM32H563VGT6, Y1 X322525MOB4SI, Y2 X322525MOB4SI

Commit message: Updated resistor naming in sch, updated manufacture files and license
Parts:
- removed C100, C102, C103, C191, C192, C281, C57, C58, C59, C60, C61, C62, C63, C64, C65, C81, C82, C86, C87, C89, C96, C97, C99: M1, Capacitor_SMD:C_0402_1005Metric
- removed C101, C188, C84, C85: 12P, Capacitor_SMD:C_0402_1005Metric
- removed C104: 1M, Capacitor_SMD:C_0402_1005Metric
- removed C189, C83, C88, C90, C91, C92: 1M, Capacitor_SMD:C_0603_1608Metric
- removed C190: 470P, Capacitor_SMD:C_0402_1005Metric
- removed C193, C194: 1N, Capacitor_SMD:C_0603_1608Metric
- removed C282, C283, C285, C286, C98: 10M, Capacitor_SMD:C_0603_1608Metric
- removed C284: 10M, Capacitor_SMD:C_0805_2012Metric
- removed C93, C94: 1P5, Capacitor_SMD:C_0402_1005Metric
- removed C95: 1N, Capacitor_SMD:C_1206_3216Metric
- removed D13, D14, D20: LED, LED_SMD:LED_0603_1608Metric
- removed D21, D24: 1N5819WS, Diode_SMD:D_SOD-323
- removed D25: SMAJ24A, Diode_SMD:D_SMA
- removed D26, D27, D36, D37, D42, D43, D44, D45: DNP, Diode_SMD:D_SOD-323
- removed F1: SMD1812P150TF/24, Fuse:Fuse_1812_4532Metric_Pad1.30x3.40mm_HandSolder
- removed FB1, FB2, FB3, FB4, FB5, FB6: GZ1608D601TF, Inductor_SMD:L_0603_1608Metric
- removed FL1: ACM2012-900-2P-T002, Inductor_SMD:L_CommonModeChoke_Coilcraft_0805USB
- removed J40: Micro_SD_Card, Connector_Card:microSD_HC_Molex_47219-2001
- removed J41: RJHSE5383, Connector_RJ:RJ45_Amphenol_RJHSE538X
- removed J42: USB_C_Receptacle_USB2.0, Connector_USB:USB_C_Receptacle_GCT_USB4105-xx-A_16P_TopMnt_Horizontal
- removed R100: 100R, Capacitor_SMD:C_0603_1608Metric
- removed R101, R113, R114, R116, R117, R118, R119, R120, R121, R279, R280, R281, R282, R323, R324: 10K, Resistor_SMD:R_0402_1005Metric
- removed R102: 0R, Capacitor_SMD:C_0603_1608Metric
- removed R103: 1M, Resistor_SMD:R_1206_3216Metric
- removed R105, R106, R107, R112: 49R9, Resistor_SMD:R_0402_1005Metric
- removed R108, R111, R276, R277, R278: 330R, Resistor_SMD:R_0402_1005Metric
- removed R115: 12K1, Resistor_SMD:R_0402_1005Metric
- removed R122, R123, R124, R283, R284, R285, R286, R287, R288, R289, R290, R291, R292, R293, R294, R295, R296, R297, R298, R299, R300, R301, R302, R303, R304, R305, R306, R307, R308, R309, R310, R311, R312, R313, R314, R315, R316, R317, R318, R319, R320, R321, R322, R325, R326, R327, R328: 33R, Resistor_SMD:R_0402_1005Metric
- removed R125, R126: 75R, Capacitor_SMD:C_0603_1608Metric
- removed R99: 100R, Resistor_SMD:R_0402_1005Metric
- removed U10: W25x_SOIC8 (DNP), Package_SO:SOIC-8_3.9x4.9mm_P1.27mm
- removed U11: W25x_WSOIC8 (DNP), Package_SO:SOIC-8_3.9x4.9mm_P1.27mm
- removed U13: LAN8720A, Package_DFN_QFN:VQFN-24-1EP_4x4mm_P0.5mm_EP2.5x2.5mm_ThermalVias
- removed U15, U16: SN74LV595APWR, Package_SO:TSSOP-16_4.4x5mm_P0.65mm
- removed U30: AP63200WU, Package_TO_SOT_SMD:TSOT-23-6
- removed U8: TL431DBZ, Resistor_SMD:R_0402_1005Metric
- removed U9: STM32H563VGT6, Package_QFP:LQFP-100_14x14mm_P0.5mm
- removed Y1, Y2: X322525MOB4SI, Crystal:Crystal_SMD_3225-4Pin_3.2x2.5mm
- added D38: LED-R-0603_KT-0603R, cm5-module-Library:LED_0603_1608Metric_R, F.Cu at (204.8, 56.2)
- added J44: ATX5V, Connector_PinHeader_2.54mm:PinHeader_1x02_P2.54mm_Vertical, F.Cu at (197.6, 144.5)
- added J45: ATX5VSB, Connector_PinHeader_2.54mm:PinHeader_1x02_P2.54mm_Vertical, F.Cu at (197.6, 137.6)
- added J46: ATX5V, Connector_PinHeader_2.54mm:PinHeader_1x02_P2.54mm_Vertical, F.Cu at (197.6, 130.8)
- added J47: ATX5VSB, Connector_PinHeader_2.54mm:PinHeader_1x02_P2.54mm_Vertical, F.Cu at (197.6, 123.9)
- added J48: PWR_JMPER, Connector_PinHeader_2.54mm:PinHeader_1x02_P2.54mm_Vertical, F.Cu at (53.9, 152.5)
- added J49: ATXPWR_JMPER, Connector_PinHeader_2.54mm:PinHeader_1x02_P2.54mm_Vertical, F.Cu at (180.0, 95.5)
- added J50: RPI_UART, Connector_PinHeader_2.54mm:PinHeader_1x04_P2.54mm_Vertical, F.Cu at (67.0, 44.2)
- added J51: JTAG_UPSTREAM_2x5, Connector_PinHeader_2.54mm:PinHeader_2x05_P2.54mm_Vertical, F.Cu at (196.0, 259.3)
- added R128: R-10k-0402, Resistor_SMD:R_0402_1005Metric_Pad0.72x0.64mm_HandSolder, F.Cu at (201.9, 56.3)
- added R129: 10K, Resistor_SMD:R_0603_1608Metric_Pad0.98x0.95mm_HandSolder, F.Cu at (186.9, 94.2)
- added R130: R-0R-0402, Resistor_SMD:R_0402_1005Metric_Pad0.72x0.64mm_HandSolder, F.Cu at (196.9, 265.9)
- BT1, C9: moved to F.Cu
- R10, R11: moved to B.Cu
- moved R14 73.8 mm to (201.4, 40.0)
- moved D17 72.7 mm to (204.6, 40.0)
- moved R15 72.7 mm to (201.5, 43.6)
- moved R110 71.9 mm to (201.7, 47.0)
- moved D18 71.6 mm to (204.6, 43.6)
- moved R2 71.1 mm to (201.9, 50.4)
- moved D2 71.1 mm to (204.7, 50.3)
- moved D19 70.6 mm to (204.6, 46.9)
- moved R1 70.0 mm to (202.0, 53.3)
- moved D1 70.0 mm to (204.7, 53.2)
- moved J19 68.7 mm to (138.2, 172.5)
- moved TP3 58.6 mm to (105.1, 53.5)
- moved TP2 56.1 mm to (106.8, 53.5)
- moved J27 53.3 mm to (131.3, 185.9)
- moved J18 43.9 mm to (151.0, 262.7)
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Connections:
- J43 pad 1: unconnected-(J43-+3.3V-Pad1) -> /ATX3V3
- J43 pad 12: unconnected-(J43-+3.3V-Pad1)_3 -> /ATX3V3
- J43 pad 13: unconnected-(J43-+3.3V-Pad1)_2 -> /ATX3V3
- J43 pad 14: unconnected-(J43--12V-Pad14) -> /ATXNeg12V
- J43 pad 16: unconnected-(J43-PS_ON#-Pad16) -> Net-(J43-PS_ON#)
- J43 pad 2: unconnected-(J43-+3.3V-Pad1)_1 -> /ATX3V3
- J43 pad 21: unconnected-(J43-+5V-Pad21)_4 -> /ATX5V
- J43 pad 22: unconnected-(J43-+5V-Pad21)_3 -> /ATX5V
- J43 pad 23: unconnected-(J43-+5V-Pad21)_2 -> /ATX5V
- J43 pad 4: unconnected-(J43-+5V-Pad21) -> /ATX5V
- J43 pad 6: unconnected-(J43-+5V-Pad21)_1 -> /ATX5V
- J43 pad 8: unconnected-(J43-PWR_OK-Pad8) -> /ATXPWROK
- J43 pad 9: unconnected-(J43-+5VSB-Pad9) -> /ATX5VSB
- J8 pad MP: (no net) -> GND
- R18 pad 1: /ISET -> /ISET_VBUS
- R37 pad 1: /ISET -> /ISET_SD3V3
- U1 pad 5: /ISET -> /ISET_VBUS
- U14 pad 14: /PCIE X8 FPGA0/TX6.+ -> /PCIE X8 FPGA0/RX6.+
- U14 pad 15: /PCIE X8 FPGA0/TX6.- -> /PCIE X8 FPGA0/RX6.-
- U14 pad 33: /PCIE X8 FPGA0/RX6.+ -> /PCIE X8 FPGA0/TX6.+
- U14 pad 34: /PCIE X8 FPGA0/RX6.- -> /PCIE X8 FPGA0/TX6.-
- U17 pad 14: /PCIE X8 FPGA1/TX6.+ -> /PCIE X8 FPGA1/RX6.+
- U17 pad 15: /PCIE X8 FPGA1/TX6.- -> /PCIE X8 FPGA1/RX6.-
- U17 pad 33: /PCIE X8 FPGA1/RX6.+ -> /PCIE X8 FPGA1/TX6.+
- U17 pad 34: /PCIE X8 FPGA1/RX6.- -> /PCIE X8 FPGA1/TX6.-
- U18 pad 14: /PCIE X8 FPGA2/TX6.+ -> /PCIE X8 FPGA2/RX6.+
- U18 pad 15: /PCIE X8 FPGA2/TX6.- -> /PCIE X8 FPGA2/RX6.-
- U18 pad 33: /PCIE X8 FPGA2/RX6.+ -> /PCIE X8 FPGA2/TX6.+
- U18 pad 34: /PCIE X8 FPGA2/RX6.- -> /PCIE X8 FPGA2/TX6.-
- U19 pad 14: /PCIE X8 FPGA3/TX6.+ -> /PCIE X8 FPGA3/RX6.+
- U19 pad 15: /PCIE X8 FPGA3/TX6.- -> /PCIE X8 FPGA3/RX6.-
- U19 pad 33: /PCIE X8 FPGA3/RX6.+ -> /PCIE X8 FPGA3/TX6.+
- U19 pad 34: /PCIE X8 FPGA3/RX6.- -> /PCIE X8 FPGA3/TX6.-
- U7 pad 5: /ISET -> /ISET_SD3V3
Routing:
- net /PWR_BTN: track 13.0 -> 224.4 mm, vias 0 -> 4
- net /FPGA1_nPRSNT: track 0.00 -> 211.0 mm, vias 0 -> 5
- net /GPIO12: track 0.00 -> 210.4 mm, vias 0 -> 1
- net /FPGA3_RST: track 0.00 -> 208.9 mm, vias 0 -> 3
- net /FPGA3_nPRSNT: track 0.00 -> 207.9 mm, vias 0 -> 6
- net /GPIO21: track 0.00 -> 207.9 mm, vias 0 -> 1
- net /GPIO20: track 0.00 -> 207.2 mm, vias 0 -> 1
- net /GPIO16: track 0.00 -> 206.3 mm, vias 0 -> 1
- net /FPGA2_nPRSNT: track 0.00 -> 202.9 mm, vias 0 -> 6
- net /FPGA2_RST: track 0.00 -> 196.9 mm, vias 0 -> 4
- net /FPGA1_RST: track 0.00 -> 196.5 mm, vias 0 -> 3
- net /FPGA0_RST: track 0.00 -> 194.3 mm, vias 0 -> 5
- net +5V: track 11.6 -> 203.2 mm, vias 1 -> 18
- net /FPGA0_nPRSNT: track 13.0 -> 193.2 mm, vias 2 -> 9
- net GND: track 235.9 -> 411.3 mm, vias 291 -> 518
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- added copper zone on B.Cu, net +12V
- added copper zone on F.Cu, net +12V
- added copper zone on In2.Cu, net +12V
- added copper zone on B.Cu, net +1V0_PCIE
- added copper zone on F.Cu, net +1V0_PCIE
- added copper zone on In2.Cu, net +3V3
- added copper zone on B.Cu, net +5V
- added copper zone on In2.Cu, net +5V
- removed copper zone on In2.Cu, net GND
Other:
- board text added: "-12V ATX3V3 5VSB ATX5V"
- board text added: "5V 12V 3.3V PWR ACT ATX PGOOD"
- board text added: "ATX JUMPER"
- board text added: "GND RPi TX RPi RX 3V3"
- board text added: "JTAG"
- board text added: "POWER"
- board text added: "PPS OUT"
- board text added: "RPi JUMPER"
- board text added: "RPi USB2"
