File: 1-baseboard/TentaLab/tentalab.kicad_sch (KiCad schematic)
At the start: 246 parts, among them J1 USB-A_USB-303WSD-BRY, J10 Micro_SD_Card, J11 RPI_HEADER, J12 RPI_OPTIONS, J13 RJ45_HC612601A-M893-A, J16 12V ATX, J17 JTAG_0, J18 JTAG_0, J19 JTAG_0, J2 JTAG_UPSTREAM, J20 Jack-DC, J21 FPGA_RST_nPRSNT, J23 RPi UART, J24 JTAG_0, J25 JTAG_SKIP_0, J26 JTAG_SKIP_0, J27 JTAG_SKIP_0, J28 JTAG_SKIP_0, J29 Conn_01x22_Female, J3 CM5_1-100_3mm-stack, J30 Conn_01x22_Female, J4 CM5_101-200_3mm-stack, J5 HDMI_A, J6 Conn_Coaxial_Small, J7 HDMI_A, J8 Conn_01x04, J9 RPi USB2, SW1 PWR_BTN, U1 AP22615AWU-7, U12 RT9742SNGV, U2 PI7C9X2G608ELBZXAE, U3 TPS62821DLC, U4 M93C86, U5 CH330N, U6 TPS563200, U7 AP22615AWU-7

Commit message: baseboard sch with qsfp, layout in progress
Parts:
- removed J29, J30: Conn_01x22_Female, CM5IOLibrary:Hirose_FH12-22S-0.5SH_1x22-1MP_P0.50mm_Horizontal, symbol Connector:Conn_01x22_Socket
- added J29, J30: Conn_01x22_Female, CM5IOLibrary:Hirose_FH12-22S-0.5SH_1x22-1MP_P0.50mm_Horizontal, symbol Connector:Conn_01x23_Socket
- added J43: ATX-24, Connector_Molex:Molex_Mini-Fit_Jr_5566-24A_2x12_P4.20mm_Vertical, symbol Connector:ATX-24
- added R127: R-2k2-0402, Resistor_SMD:R_0402_1005Metric_Pad0.72x0.64mm_HandSolder, symbol DW-resistors:R-2k2-0402
- D22, D23: footprint DW-footprints:SOT1176-1 -> cm5-module-Library:SOT1176-1
Connections:
- net +12V: now also J43.10 (+12V), J43.11 (+12V)
- net +3V3: now also J29.22 (Pin_22), J30.22 (Pin_22)
- net +5V: now also R127.2
- net AGND: now also J10.SH1, J10.SH2, J10.SH3, J10.SH4, J29.1 (Pin_1), J29.10 (Pin_10), J29.13 (Pin_13), J29.16 (Pin_16), J29.19 (Pin_19), J29.23 (Pin_23), J29.4 (Pin_4), J29.7 (Pin_7), J30.1 (Pin_1), J30.10 (Pin_10), J30.13 (Pin_13), J30.16 (Pin_16), J30.19 (Pin_19), J30.23 (Pin_23), J30.4 (Pin_4), J30.7 (Pin_7), J43.15 (GND), J43.17 (GND), J43.18 (GND), J43.19 (GND), J43.24 (GND), J43.3 (GND), J43.5 (GND), J43.7 (GND); no longer J10.9 (SHIELD)
- net CAM_GPIO0: now also J29.17 (Pin_17)
- net CAM_GPIO1: now also J29.18 (Pin_18)
- net ID_SC: now also J30.20 (Pin_20)
- net ID_SD: now also J30.21 (Pin_21)
- net MIPI_0.CLK+: now also J29.9 (Pin_9)
- net MIPI_0.CLK-: now also J29.8 (Pin_8)
- net MIPI_0.D0+: now also J29.3 (Pin_3)
- net MIPI_0.D0-: now also J29.2 (Pin_2)
- net MIPI_0.D1+: now also J29.6 (Pin_6)
- net MIPI_0.D1-: now also J29.5 (Pin_5)
- net MIPI_0.D2+: now also J29.12 (Pin_12)
- net MIPI_0.D2-: now also J29.11 (Pin_11)
- net MIPI_0.D3+: now also J29.15 (Pin_15)
- net MIPI_0.D3-: now also J29.14 (Pin_14)
- net MIPI_1.CLK+: now also J30.9 (Pin_9)
- net MIPI_1.CLK-: now also J30.8 (Pin_8)
- net MIPI_1.D0+: now also J30.3 (Pin_3)
- net MIPI_1.D0-: now also J30.2 (Pin_2)
- net MIPI_1.D1+: now also J30.6 (Pin_6)
- net MIPI_1.D1-: now also J30.5 (Pin_5)
- net MIPI_1.D2+: now also J30.12 (Pin_12)
- net MIPI_1.D2-: now also J30.11 (Pin_11)
- net MIPI_1.D3+: now also J30.15 (Pin_15)
- net MIPI_1.D3-: now also J30.14 (Pin_14)
- net PCIE_SCL: now also J29.20 (Pin_20)
- net PCIE_SDA: now also J29.21 (Pin_21)
- net REFCLK1_PIN+: now reaches C14.2, U2.AR21 (REFCLKN[0])
- net REFCLKO5_PIN-: now reaches R65.1, U2.AA35 (REFCLKON[5])
- net REFCLKO3_PIN+: now reaches R60.1, U2.P34 (REFCLKOP[3])
- net RPiUSB2_VBUS: now reaches C7.1, C8.1, J9.A4 (VBUS), J9.A9 (VBUS), J9.B4 (VBUS), J9.B9 (VBUS), R89.2, R9.1
- net REFCLK2_PIN+: now reaches C17.2, U2.A19 (REFCLKN[1])
- net REFCLK2_PIN-: now reaches C16.2, U2.A21 (REFCLKP[1])
- net REFCLKO7_PIN+: now reaches R66.1, U2.AB34 (REFCLKOP[7])
- net REFCLKO7_PIN-: now reaches R67.1, U2.AD34 (REFCLKON[7])
- net REFCLK1_PIN-: now reaches C15.2, U2.AR19 (REFCLKP[0])
- net REFCLKO1_PIN+: now reaches R56.1, U2.K34 (REFCLKOP[1])
- net REFCLKO2_PIN+: now reaches R58.1, U2.L35 (REFCLKOP[2])
- net REFCLKO1_PIN-: now reaches R57.1, U2.M34 (REFCLKON[1])
- net REFCLKO2_PIN-: now reaches R59.1, U2.N35 (REFCLKON[2])
- net REFCLKO3_PIN-: now reaches R61.1, U2.R35 (REFCLKON[3])
- net PCIe.REFCLK_PIN+: now reaches C106.2, U2.T34 (REFCLKIP)
- net PCIe.REFCLK_PIN-: now reaches C105.2, U2.U35 (REFCLKIN)
- net REFCLKO4_PIN+: now reaches R62.1, U2.V34 (REFCLKOP[4])
- net REFCLKO4_PIN-: now reaches R63.1, U2.W35 (REFCLKON[4])
- net REFCLKO5_PIN+: now reaches R64.1, U2.Y34 (REFCLKOP[5])
- net at U1.3 (~{FLG}): now also R127.1
- net RPiUART_VBUS: now reaches C79.2, J23.A4 (VBUS), J23.A9 (VBUS), J23.B4 (VBUS), J23.B9 (VBUS), U5.5 (VCC)
- net at R171.2: now also J30.17 (Pin_17)
- net REFCLKO1+ renamed REFCLKO1.+
- net REFCLKO1- renamed REFCLKO1.-
- net REFCLKO2+ renamed REFCLKO2.+
- net REFCLKO2- renamed REFCLKO2.-
- net REFCLKO3+ renamed REFCLKO3.+
- net REFCLKO3- renamed REFCLKO3.-
- net REFCLKO4+ renamed REFCLKO4.+
- net REFCLKO4- renamed REFCLKO4.-
- net REFCLKO5+ renamed REFCLKO5.+
- net REFCLKO5- renamed REFCLKO5.-
- net REFCLKO7+ renamed REFCLKO7.+
- net REFCLKO7- renamed REFCLKO7.-
- new net: J43.1 (+3.3V), J43.12 (+3.3V), J43.13 (+3.3V), J43.2 (+3.3V)
- new net: J43.21 (+5V), J43.22 (+5V), J43.23 (+5V), J43.4 (+5V), J43.6 (+5V)
- no-connect marks 64 -> 52
Other:
- added sheet QSFP1 (qsfp.kicad_sch)
- added sheet QSFP2 (qsfp.kicad_sch)
- added sheet QSFP3 (qsfp.kicad_sch)
- added sheet QSFP4 (qsfp.kicad_sch)
- added sheet SMU (H5_Management_Mod.kicad_sch)
- note added: "5V derived from 12V IN, jack, ATX 6-pin, or ATX 24-pin (normal operation)"
- note added: "Reference Designs Compact design (MIT-licensed): https://github.com/Dominik-Workshop/moducard-cm5-module Official KiCad baseboard: https://pip.raspberrypi.com/categories/1098-design-files QSFP footprint (GPL v3): https://github.com/mwrnd/KiCad_Libraries Designed by Yimin Gu https://github.com/regymm Colaborate with Petr Pavlata Project URL: RPCIe TentaLab Funding: NLnet NGI0 Commons Fund https://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"
- note added: "STM32 Remote Management"
- note removed: "5V derived from 12V IN, jack or ATX 6-pin (normal operation)"
- note removed: "Reference Designs Compact design (MIT-licensed): https://github.com/Dominik-Workshop/moducard-cm5-module Official KiCad baseboard: https://pip.raspberrypi.com/categories/1098-design-files Designed by https://github.com/regymm Colaborate with Project URL: RPCIe TentaLab Funding:"
- moved on the sheet: C1, C105, C106, C14, C15, C16, C17, C18, C19, C2, C20, C21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
