File: 1-baseboard/TentaLab/tentalab.kicad_sch (KiCad schematic)
At the start: 248 parts, among them J1 USB-A_USB-303WSD-BRY, J10 Micro_SD_Card, J11 RPI_HEADER, J12 RPI_OPTIONS, J13 RJ45_HC612601A-M893-A, J16 12V ATX, J17 JTAG_0, J18 JTAG_0, J19 JTAG_0, J2 JTAG_UPSTREAM, J20 Jack-DC, J21 FPGA_RST_nPRSNT, J23 RPi UART, J24 JTAG_0, J25 JTAG_SKIP_0, J26 JTAG_SKIP_0, J27 JTAG_SKIP_0, J28 JTAG_SKIP_0, J29 Conn_01x22_Female, J3 CM5_1-100_3mm-stack, J30 Conn_01x22_Female, J4 CM5_101-200_3mm-stack, J43 ATX-24, J5 HDMI_A, J6 Conn_Coaxial_Small, J7 HDMI_A, J8 Conn_01x04, J9 RPi USB2, SW1 PWR_BTN, U1 AP22615AWU-7, U12 RT9742SNGV, U2 PI7C9X2G608ELBZXAE, U3 TPS62821DLC, U4 M93C86, U5 CH330N, U6 TPS563200, U7 AP22615AWU-7

Commit message: Updated resistor naming in sch, updated manufacture files and license
Parts:
- removed R21, R24, R25, R26, R27, R28, R33, R34, R35, R38, R39, R40, R41, R42, R56, R57, R58, R59, R60, R61, R62, R63, R64, R65, R66, R67, R68, R69, R70, R71, R72, R73, R74, R75, R76, R77, R78, R79: R-0R-0402, Resistor_SMD:R_0402_1005Metric_Pad0.72x0.64mm_HandSolder, symbol DW-resistors:R-0R-0402
- added D38: LED-R-0603_KT-0603R, cm5-module-Library:LED_0603_1608Metric_R, symbol DW-diodes:LED-R-0603_KT-0603R
- added J44, J46: ATX5V, Connector_PinHeader_2.54mm:PinHeader_1x02_P2.54mm_Vertical, symbol Connector:Conn_01x02_Pin
- added J45, J47: ATX5VSB, Connector_PinHeader_2.54mm:PinHeader_1x02_P2.54mm_Vertical, symbol Connector:Conn_01x02_Pin
- added J48: PWR_JMPER, Connector_PinHeader_2.54mm:PinHeader_1x02_P2.54mm_Vertical, symbol Connector:Conn_01x02_Pin
- added J49: ATXPWR_JMPER, Connector_PinHeader_2.54mm:PinHeader_1x02_P2.54mm_Vertical, symbol Connector:Conn_01x02_Pin
- added J50: RPI_UART, Connector_PinHeader_2.54mm:PinHeader_1x04_P2.54mm_Vertical, symbol Connector_Generic:Conn_01x04
- added J51: JTAG_UPSTREAM_2x5, Connector_PinHeader_2.54mm:PinHeader_2x05_P2.54mm_Vertical, symbol Connector_Generic:Conn_02x05_Odd_Even
- added R128: R-10k-0402, Resistor_SMD:R_0402_1005Metric_Pad0.72x0.64mm_HandSolder, symbol DW-resistors:R-10k-0402
- added R129: 10K, Resistor_SMD:R_0603_1608Metric_Pad0.98x0.95mm_HandSolder, symbol Device:R
- added R130: R-0R-0402, Resistor_SMD:R_0402_1005Metric_Pad0.72x0.64mm_HandSolder, symbol DW-resistors:R-0R-0402
- added R21, R24, R25, R26, R27, R28, R33, R34, R35, R38, R39, R40, R41, R42: 330, Resistor_SMD:R_0402_1005Metric_Pad0.72x0.64mm_HandSolder, symbol DW-resistors:330
- added R56, R57, R58, R59, R60, R61, R62, R63, R64, R65, R66, R67: 33, Resistor_SMD:R_0402_1005Metric_Pad0.72x0.64mm_HandSolder, symbol DW-resistors:33
- added R68, R69, R70, R71, R72, R73, R74, R75, R76, R77, R78, R79: 49.9, Resistor_SMD:R_0402_1005Metric_Pad0.72x0.64mm_HandSolder, symbol DW-resistors:49.9
- R127: value R-2k2-0402 -> R-10k-0402
- R16, R19: value R-0R-0402 -> 1.43K
- R20: value R-0R-0402 -> 475
- R22, R23: value R-0R-0402 -> 330
- R29, R31, R8: value R-10k-0402 -> 5.1K
- R3: value R-10k-0402 -> 5.1k
- R32: value R-0R-0402 -> 1K
- R43: value R-0R-0402 -> 475R
- R45, R47, R49, R51, R53, R55: value R-0R-0402 -> 10k
- R6: value R-0R-0402 -> 5.1K
- R80: value R-10k-0402 -> 180k
- R81: value R-10k-0402 -> 120k
- R82: value R-10k-0402 -> 0
Connections:
- net +3V3: now also J50.4 (Pin_4), R130.1
- net AGND: now also J8.MP, J44.2 (Pin_2), J45.2 (Pin_2), J46.2 (Pin_2), J47.2 (Pin_2), J48.2 (Pin_2), J49.2 (Pin_2), J50.1 (Pin_1), J51.10 (Pin_10), R128.1, R129.2, R21.1, R24.1, R25.1, R26.1, R27.1, R28.1, R33.1, R34.1, R35.1, R38.1, R39.1, R40.1, R41.1, R42.1, R68.2, R69.2, R70.2, R71.2, R72.2, R73.2, R74.2, R75.2, R76.2, R77.2, R78.2, R79.2
- net GPIO4: now also J50.2 (Pin_2)
- net GPIO5: now also J50.3 (Pin_3)
- net JTAG_SRST: now also J51.6 (Pin_6)
- net JTAG_TCK: now also J51.1 (Pin_1)
- net JTAG_TDI: now also J51.9 (Pin_9)
- net JTAG_TDO: now also J51.3 (Pin_3)
- net JTAG_TMS: now also J51.5 (Pin_5)
- net PWR_BTN: now also J48.1 (Pin_1)
- net REFCLKO1.+: now also R56.2, R68.1
- net REFCLKO1.-: now also R57.2, R69.1
- net REFCLKO1_PIN+: now also R56.1
- net REFCLKO1_PIN-: now also R57.1
- net REFCLKO2.+: now also R58.2, R70.1
- net REFCLKO2.-: now also R59.2, R71.1
- net REFCLKO2_PIN+: now also R58.1
- net REFCLKO2_PIN-: now also R59.1
- net REFCLKO3.+: now also R60.2, R72.1
- net REFCLKO3.-: now also R61.2, R73.1
- net REFCLKO3_PIN+: now also R60.1
- net REFCLKO3_PIN-: now also R61.1
- net REFCLKO4.+: now also R62.2, R74.1
- net REFCLKO4.-: now also R63.2, R75.1
- net REFCLKO4_PIN+: now also R62.1
- net REFCLKO4_PIN-: now also R63.1
- net REFCLKO5.+: now also R64.2, R76.1
- net REFCLKO5.-: now also R65.2, R77.1
- net REFCLKO5_PIN+: now also R64.1
- net REFCLKO5_PIN-: now also R65.1
- net REFCLKO7.+: now also R66.2, R78.1
- net REFCLKO7.-: now also R67.2, R79.1
- net REFCLKO7_PIN+: now also R66.1
- net REFCLKO7_PIN-: now also R67.1
- net at U2.W1 (PL_512B/DBO[0]): now also R28.2
- net ATX3V3: now reaches J43.1 (+3.3V), J43.12 (+3.3V), J43.13 (+3.3V), J43.2 (+3.3V)
- net ATX3V3: now also J46.1 (Pin_1)
- net ATXNeg12V: now reaches J43.14 (-12V)
- net ATXNeg12V: now also J47.1 (Pin_1)
- net at J43.16 (PS_ON#): now also J49.1 (Pin_1), R129.1
- net ATX5V: now reaches J43.21 (+5V), J43.22 (+5V), J43.23 (+5V), J43.4 (+5V), J43.6 (+5V)
- net ATX5V: now also J44.1 (Pin_1)
- net ATXPWROK: now reaches J43.8 (PWR_OK)
- net ATXPWROK: now also D38.2 (A)
- net ATX5VSB: now reaches J43.9 (+5VSB)
- net ATX5VSB: now also J45.1 (Pin_1)
- net at U2.K2 (GPIO[2]): now also R35.2
- net at U2.AB2 (UPS_PORTSEL[0]/DBO[3]): now also R24.2
- net at U2.AE1 (UPS_PORTSEL[1]/DBO[4]): now also R25.2
- net at U2.AF2 (UPS_PORTSEL[2]): now also R26.2
- net at U2.AG1 (UPS_PORTSEL[3]): now also R27.2
- net at U2.AH2 (CLKBUF_PD): now also R21.2
- net at U2.H2 (GPIO[0]): now also R33.2
- net at U2.J1 (GPIO[1]): now also R34.2
- net at U2.L1 (GPIO[3]): now also R38.2
- net at U2.P2 (GPIO[4]): now also R39.2
- net at U2.R1 (GPIO[5]): now also R40.2
- net at U2.T2 (GPIO[6]): now also R41.2
- net at U2.U1 (GPIO[7]): now also R42.2
- net ISET renamed ISET_SD3V3
- net ISET_SD3V3: no longer R18.1, U1.5 (ISET)
- new net: J51.4 (Pin_4), R130.2
- new net: D38.1 (C), R128.2
- new net ISET_VBUS: R18.1, U1.5 (ISET)
- no-connect marks 52 -> 50
Other:
- note added: "Planned to operate externally"
- note added: "Reference Designs Compact design (MIT-licensed): https://github.com/Dominik-Workshop/moducard-cm5-module Official KiCad baseboard: https://pip.raspberrypi.com/categories/1098-design-files QSFP footprint (GPL v3): https://github.com/mwrnd/KiCad_Libraries Designed by Yimin Gu https://github.com/regymm Colaborate with Petr Pavlata https://www.linkedin.com/in/acrux-systems/ Project URL: RPCIe TentaLa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"
- note removed: "Reference Designs Compact design (MIT-licensed): https://github.com/Dominik-Workshop/moducard-cm5-module Official KiCad baseboard: https://pip.raspberrypi.com/categories/1098-design-files QSFP footprint (GPL v3): https://github.com/mwrnd/KiCad_Libraries Designed by Yimin Gu https://github.com/regymm Colaborate with Petr Pavlata Project URL: RPCIe TentaLab Funding: NLnet NGI0 Commons Fund https://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"
- moved on the sheet: D15, D16, D17, D18, D19, J20, J43, R110, R12, R13, R14, R15
