File: 1-baseboard/TentaLab/sfp.kicad_sch (KiCad schematic)
At the start: 27 parts, among them J31 SFP+

Commit message: Updated resistor naming in sch, updated manufacture files and license
Parts:
- R172, R183: value R-10k-0402 -> 0.1R
- R173, R184: value R-10k-0402 -> 0.5R
